File: schema-ontwerp/oppakkerV3/oppakkerV4.kicad_sch (KiCad schematic)
At the start: 25 parts, among them J1 Conn_01x03, J2 Conn_01x03, J3 Conn_01x02, J6 Conn_01x04, Q1 IRLB8721PBF, Q2 IRLB8721PBF, Q3 IRLB8721PBF, Q4 IRLB8721PBF, SW1 SW_Push

Commit message: update
Parts:
- removed J1, J2: Conn_01x03, Connector_Molex:Molex_KK-254_AE-6410-03A_1x03_P2.54mm_Vertical, symbol Connector_Generic:Conn_01x03
- added J1, J4: Conn_01x04, TerminalBlock:TerminalBlock_MaiXu_MX126-5.0-04P_1x04_P5.00mm, symbol Connector_Generic:Conn_01x04
- C2: value C_Polarized -> 470uF; footprint Capacitor_THT:CP_Axial_L10.0mm_D4.5mm_P15.00mm_Horizontal -> Capacitor_THT:C_Disc_D3.0mm_W1.6mm_P2.50mm
- D1, D2, D3, D4: footprint Diode_THT:D_A-405_P2.54mm_Vertical_AnodeUp -> Resistor_THT:R_Axial_DIN0204_L3.6mm_D1.6mm_P7.62mm_Horizontal
- J3: footprint Connector_Molex:Molex_KK-254_AE-6410-02A_1x02_P2.54mm_Vertical -> TerminalBlock:TerminalBlock_MaiXu_MX126-5.0-02P_1x02_P5.00mm
Connections:
- net +48V: now also J1.2 (Pin_2), J1.4 (Pin_4), J4.2 (Pin_2), J4.4 (Pin_4)
- net at A1.10 (D7): now also R2.2; no longer BZ1.1 (+)
- net at A1.5 (D2): now also BZ1.1 (+); no longer R2.2
- net at A1.6 (D3): now also R7.2; no longer R5.2
- net at A1.8 (D5): now also R5.2; no longer R7.2
- net at D3.2 (A), Q1.2 (D): now also J4.3 (Pin_3)
- net at D2.2 (A), Q2.2 (D): now also J4.1 (Pin_1)
- net at D1.2 (A), Q3.2 (D): now also J1.1 (Pin_1)
- net at D4.2 (A), Q4.2 (D): now also J1.3 (Pin_3)
